File: 6502 PCB.kicad_pcb (KiCad board)
At the start: 2 copper layers, 25 parts, among them SW1 RESET, SW2 SW_Push, SW3 SW_Push, SW4 SW_Push, SW5 SW_Push, SW6 SW_Push, U1 W65C02S, U2 28C256, U3 62256, U4 W65C22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

Commit message: bumb
Parts:
- DS1: footprint Display:HY1602E -> Display:WC1602A
- moved DS1 220.6 mm to (27.9, 87.9)
- moved U2 90.1 mm to (22.9, 53.3), turned to 90 degrees
- moved SW4 69.8 mm to (147.3, 104.1)
- moved SW1 68.2 mm to (27.9, 25.4)
- moved X1 65.9 mm to (63.5, 27.9)
- moved C4 64.3 mm to (125.5, 37.9)
- moved C2 64.3 mm to (125.5, 28.2)
- moved C3 64.3 mm to (125.5, 33.0)
- moved R1 64.3 mm to (130.1, 29.8)
- moved R2 64.3 mm to (130.1, 31.6)
- moved R3 64.3 mm to (130.1, 33.3)
- moved R4 64.3 mm to (130.1, 35.1)
- moved R5 64.3 mm to (130.1, 36.8)
- moved R6 64.3 mm to (130.1, 38.6)
- moved R7 64.3 mm to (130.1, 40.3)
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
Commit message: Add files via upload
Parts:
- removed C2, C3, C4: 0.1uf, Capacitor_SMD:CP_Elec_3x5.3
- added J1: power_source, TerminalBlock:TerminalBlock_Altech_AK300-2_P5.00mm, F.Cu at (17.8, 20.3)
- DS1: value HY1602E -> HD44780U
- R1, R2, R3, R4, R5, R6, R7: footprint Resistor_SMD:R_0201_0603Metric -> Resistor_SMD:R_0201_0603Metric_Pad0.64x0.40mm_HandSolder
- moved C1 33.0 mm to (113.3, 53.3)
- moved U5 31.1 mm to (66.0, 21.6)
- moved RV1 27.2 mm to (101.6, 73.7)
- moved X1 20.7 mm to (43.2, 24.1)
- moved DS1 17.8 mm to (21.9, 71.1)
- moved U4 14.4 mm to (53.3, 66.0)
- moved U1 12.7 mm to (53.3, 45.7)
- moved U3 12.7 mm to (15.2, 66.0)
- moved R1 11.7 mm to (141.8, 30.3)
- moved R2 11.7 mm to (141.8, 32.1)
- moved R3 11.7 mm to (141.8, 33.8)
- moved R4 11.7 mm to (141.8, 35.6)
- moved R5 11.7 mm to (141.8, 37.3)
- moved R6 11.7 mm to (141.8, 39.1)
- moved R7 11.7 mm to (141.8, 40.8)
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Connections:
- C1 pad 2: GND -> /GND
- DS1 pad 1: GND -> /GND
- DS1 pad 15: GND -> /GND
- DS1 pad 16: +5V -> /VDD
- DS1 pad 2: +5V -> /VDD
- R1 pad 1: +5V -> /VDD
- R2 pad 1: +5V -> /VDD
- R3 pad 1: +5V -> Net-(U4-PA0)
- R3 pad 2: Net-(U4-PA0) -> /VDD
- R4 pad 1: +5V -> Net-(U4-PA1)
- R4 pad 2: Net-(U4-PA1) -> /VDD
- R5 pad 1: +5V -> Net-(U4-PA2)
- R5 pad 2: Net-(U4-PA2) -> /VDD
- R6 pad 1: +5V -> Net-(U4-PA3)
- R6 pad 2: Net-(U4-PA3) -> /VDD
- R7 pad 1: +5V -> Net-(U4-PA4)
- R7 pad 2: Net-(U4-PA4) -> /VDD
- RV1 pad 1: GND -> /GND
- SW1 pad 1: GND -> Net-(U1-~{RES})
- SW1 pad 2: Net-(U1-~{RES}) -> /GND
- SW2 pad 2: GND -> /GND
- SW3 pad 2: GND -> /GND
- SW4 pad 2: GND -> /GND
- SW5 pad 2: GND -> /GND
- SW6 pad 2: GND -> /GND
- U1 pad 21: GND -> /GND
- U1 pad 36: +5V -> /VDD
- U1 pad 6: +5V -> /VDD
- U1 pad 8: +5V -> /VDD
- U2 pad 14: GND -> /GND
- U2 pad 22: GND -> /GND
- U2 pad 27: +5V -> /VDD
- U2 pad 28: +5V -> /VDD
- U3 pad 14: GND -> /GND
- U3 pad 22: GND -> /GND
- U3 pad 27: +5V -> /VDD
- U3 pad 28: +5V -> /VDD
- U4 pad 1: GND -> /GND
- U4 pad 20: +5V -> /VDD
- X1 pad 14: +5V -> /VDD
- X1 pad 7: GND -> /GND
Routing:
- net /VDD: track 0.00 -> 245.6 mm
- net /GND: track 0.00 -> 37.7 mm

Commit message: Add files via upload
almost done with pcb design
Parts:
- moved R1 112.8 mm to (30.0, 15.2)
- moved R2 91.9 mm to (53.8, 58.4)
- moved R3 55.2 mm to (89.3, 16.8)
- moved R4 55.2 mm to (89.3, 18.6)
- moved R5 55.2 mm to (89.3, 20.3)
- moved R6 55.2 mm to (89.3, 22.1)
- moved R7 55.2 mm to (89.3, 23.8)
- moved C1 18.5 mm to (95.5, 58.4)
- moved RV1 17.8 mm to (103.5, 91.3)
- moved DS1 17.8 mm to (23.9, 88.8)
- moved U3 17.8 mm to (17.2, 83.7)
- moved U4 17.8 mm to (55.3, 83.7)
- moved SW4 9.56 mm to (137.8, 104.3)
- moved SW3 7.62 mm to (104.1, 104.1)
- moved SW2 7.62 mm to (121.9, 104.1)
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Routing:
- net /GND: track 37.7 -> 180.4 mm, vias 0 -> 1
- net /a3: track 0.00 -> 97.1 mm
- net /a14: track 0.00 -> 94.2 mm, vias 0 -> 1
- net /a12: track 0.00 -> 92.5 mm
- net /a13: track 0.00 -> 80.2 mm
- net /a11: track 0.00 -> 80.0 mm, vias 0 -> 1
- net /a9: track 0.00 -> 77.4 mm
- net /a8: track 0.00 -> 77.4 mm
- net /a7: track 0.00 -> 75.9 mm
- net /a10: track 0.00 -> 72.4 mm
- net /a6: track 0.00 -> 70.4 mm
- net /a5: track 0.00 -> 65.0 mm
- net /a4: track 0.00 -> 59.5 mm
- net /d7: track 0.00 -> 54.4 mm
- net /VDD: track 245.6 -> 195.8 mm, vias 0 -> 3
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
Commit message: Add files via upload
redid pretty much everything
Parts:
- moved R1 177.3 mm to (188.4, 95.0)
- moved SW1 175.6 mm to (202.4, 69.3)
- moved R2 139.9 mm to (188.4, 96.8)
- moved X1 138.4 mm to (155.5, 105.1)
- moved R3 128.4 mm to (188.4, 98.5)
- moved R4 128.4 mm to (188.4, 100.3)
- moved R5 128.4 mm to (188.4, 102.0)
- moved R6 128.4 mm to (188.4, 103.8)
- moved R7 128.4 mm to (188.4, 105.5)
- moved U5 121.1 mm to (187.2, 21.3), turned to 0 degrees
- moved C1 104.9 mm to (193.1, 96.6)
- moved SW3 100.1 mm to (202.4, 85.0)
- moved SW2 84.9 mm to (202.4, 77.1)
- moved SW5 81.8 mm to (202.4, 100.7)
- moved SW6 81.6 mm to (202.4, 108.5)
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Routing:
- net /VDD: track 195.8 -> 0.00 mm, vias 3 -> 0
- net /GND: track 180.4 -> 0.15 mm, vias 1 -> 0
- net /d6: track 48.9 -> 156.7 mm, vias 0 -> 1
- net /d5: track 43.5 -> 141.6 mm, vias 0 -> 1
- net /a7: track 75.9 -> 169.8 mm
- net /a6: track 70.4 -> 158.8 mm
- net /d7: track 54.4 -> 141.1 mm, vias 0 -> 1
- net /d4: track 38.0 -> 124.7 mm, vias 0 -> 1
- net /a5: track 65.0 -> 147.9 mm
- net /d3: track 32.6 -> 110.9 mm, vias 0 -> 1
- net /d2: track 36.8 -> 114.6 mm, vias 0 -> 1
- net /a4: track 59.5 -> 136.4 mm
- net /d1: track 36.8 -> 111.9 mm, vias 0 -> 1
- net /d0: track 36.8 -> 110.9 mm, vias 0 -> 1
- net /a13: track 80.2 -> 147.6 mm
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
Commit message: Add files via upload
Parts:
- moved U5 154.3 mm to (33.0, 26.7), turned to 90 degrees
- moved R1 151.7 mm to (56.3, 20.3)
- moved SW1 144.1 mm to (66.0, 22.9)
- moved R2 142.1 mm to (53.7, 51.4)
- moved X1 106.2 mm to (83.8, 26.7)
- moved SW6 98.3 mm to (104.1, 107.3)
- moved SW2 90.7 mm to (116.8, 107.3)
- moved R7 89.1 mm to (99.5, 99.7)
- moved SW5 87.2 mm to (116.8, 117.5)
- moved SW3 86.4 mm to (116.8, 97.1)
- moved RV1 75.4 mm to (115.1, 61.0)
- moved SW4 74.3 mm to (129.5, 107.3)
- moved R3 70.6 mm to (119.8, 81.9)
- moved R4 56.4 mm to (135.8, 80.0)
- moved R5 56.4 mm to (135.8, 81.7)
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Connections:
- U5 pad 14: (no net) -> /VDD
- U5 pad 7: (no net) -> /GND
Routing:
- net /GND: track 0.15 -> 632.1 mm, vias 0 -> 2
- net /VDD: track 0.00 -> 325.0 mm, vias 0 -> 3
- net Net-(U4-PA4): track 0.00 -> 225.8 mm
- net Net-(U4-~{CS2}): track 0.00 -> 165.8 mm
- net Net-(U1-ϕ0): track 0.00 -> 127.0 mm
- net Net-(U3-~{CS}): track 0.00 -> 105.3 mm, vias 0 -> 1
- net Net-(U1-~{RES}): track 0.00 -> 94.5 mm, vias 0 -> 4
- net /a15: track 0.00 -> 93.3 mm
- net Net-(DS1-RS): track 0.00 -> 62.0 mm
- net /a14: track 134.6 -> 195.5 mm, vias 0 -> 1
- net Net-(U1-R/~{W}): track 0.00 -> 58.8 mm
- net Net-(DS1-E): track 0.00 -> 53.3 mm
- net Net-(U1-~{IRQ}): track 0.00 -> 52.3 mm
- net Net-(DS1-D7): track 0.00 -> 49.0 mm
- net Net-(DS1-D3): track 0.00 -> 48.2 mm
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
Commit message: lets gooso
Parts:
- moved C1 94.4 mm to (64.5, 20.3)
- moved RV1 94.3 mm to (23.6, 83.8)
- moved R6 39.9 mm to (99.1, 99.1), turned to 90 degrees
- moved R5 38.3 mm to (101.6, 99.1), turned to 90 degrees
- moved R4 36.9 mm to (104.1, 99.1), turned to 90 degrees
- moved R3 21.9 mm to (106.7, 99.5), turned to 90 degrees
- moved SW1 7.62 mm to (73.7, 22.9)
- moved R7 2.95 mm to (96.5, 99.5), turned to 90 degrees
Routing:
- net Net-(U4-PA1): track 0.00 -> 301.5 mm
- net Net-(U4-PA0): track 0.00 -> 289.0 mm
- net Net-(U4-PA2): track 0.00 -> 265.3 mm
- net Net-(U4-PA3): track 0.00 -> 234.0 mm
- net /VDD: track 325.0 -> 444.6 mm
- net /GND: track 632.1 -> 579.0 mm
- net Net-(DS1-V0): track 0.00 -> 28.8 mm, vias 0 -> 1
- net Net-(U1-~{RES}): track 94.5 -> 109.8 mm
- net Net-(U4-PA4): track 225.8 -> 214.0 mm
- net Net-(DS1-RS): track 62.0 -> 56.6 mm
- net Net-(DS1-D7): track 49.0 -> 48.2 mm
Other:
- board outline added: 132.1 x 124.5 mm
- board text added: "6502 8-bit Computer"
- board text added: "Created by: Joseph Hanger"

Commit message: pretty much done
Parts:
- removed DS1: HD44780U, Display:WC1602A
- removed R4, R5, R6, R7: 1K, Resistor_SMD:R_0201_0603Metric_Pad0.64x0.40mm_HandSolder
- removed RV1: 10K, Potentiometer_SMD:Potentiometer_ACP_CA6-VSMD_Vertical
- removed SW2, SW3, SW4, SW5, SW6: SW_Push, Button_Switch_SMD:SW_SPST_PTS645
- added D1: LED, LED_SMD:LED_0201_0603Metric_Pad0.64x0.40mm_HandSolder, F.Cu at (58.0, 22.9)
- added J2: Conn_01x08_Pin, Connector_PinHeader_1.00mm:PinHeader_1x08_P1.00mm_Vertical, F.Cu at (64.0, 83.8)
- added J3: Conn_01x08_Pin, Connector_PinHeader_1.00mm:PinHeader_1x08_P1.00mm_Vertical, F.Cu at (84.4, 83.8)
- C1: footprint Capacitor_SMD:CP_Elec_3x5.3 -> Capacitor_SMD:C_0201_0603Metric_Pad0.64x0.40mm_HandSolder
- moved R3 88.2 mm to (63.1, 22.9), turned to 0 degrees
Connections:
- R3 pad 1: Net-(U4-PA0) -> Net-(D1-K)
- R3 pad 2: /VDD -> /GND
- U4 pad 2: Net-(U4-PA0) -> Net-(J2-Pin_1)
- U5 pad 14: /VDD -> (no net)
- U5 pad 7: /GND -> (no net)
Routing:
- net Net-(J2-Pin_2): track 301.5 -> 8.23 mm
- net Net-(U4-PA0): track 289.0 -> 0.00 mm
- net /GND: track 579.0 -> 320.2 mm
- net Net-(J2-Pin_3): track 265.3 -> 7.59 mm
- net Net-(J2-Pin_4): track 234.0 -> 7.12 mm
- net Net-(J2-Pin_5): track 214.0 -> 8.23 mm
- net /VDD: track 444.6 -> 315.3 mm, vias 3 -> 2
- net Net-(J2-Pin_8): track 56.6 -> 9.67 mm
- net Net-(J2-Pin_6): track 53.3 -> 8.39 mm
- net Net-(J3-Pin_4): track 48.2 -> 7.12 mm
- net Net-(J3-Pin_3): track 48.2 -> 7.53 mm
- net Net-(J3-Pin_5): track 48.2 -> 7.76 mm
- net Net-(J3-Pin_2): track 48.2 -> 8.17 mm
- net Net-(J3-Pin_6): track 48.2 -> 8.39 mm
- net Net-(J2-Pin_7): track 48.2 -> 9.03 mm
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Other:
- board size 132.1 x 124.5 mm -> 132.1 x 83.8 mm
- board text added: "Inputs"
- board text added: "Outputs"

Commit message: Add files via upload
Connections:
- U5 pad 14: (no net) -> /VDD
- U5 pad 7: (no net) -> /GND
Routing:
- net /a0: track 102.2 -> 93.0 mm
- net /VDD: track 315.3 -> 309.2 mm
- added copper zone on B.Cu, net /GND
- added copper zone on F.Cu, net /GND
Other:
- board size 132.1 x 83.8 mm -> 111.8 x 83.8 mm
- board text added: "28C256"
- board text added: "62256"
- board text added: "74HC00"
- board text added: "W65C02S"
- board text added: "W65C22"
- board text added: "inputs"
- board text added: "outputs"
- board text removed: "6502 8-bit Computer"
- board text removed: "Created by: Joseph Hanger"
- board text removed: "Inputs"
- board text removed: "Outputs"
