File: 6502 PCB.kicad_sch (KiCad schematic)
At the start: 9 parts, among them SW1 RESET, U1 W65C02SxP, U2 28C256, U3 CY62256-70PC, U4 W65C22NxP, X1 1MHz

Commit message: think i finished schematic
Parts:
- added C2, C3, C4: 0.1uf, Capacitor_SMD:CP_Elec_3x5.3, symbol Device:C
- added DS1: HY1602E, Display:HY1602E, symbol Display_Character:HY1602E
- added R3, R4, R5, R6, R7: 1K, Resistor_SMD:R_0201_0603Metric, symbol Device:R
- added RV1: 10K, Potentiometer_SMD:Potentiometer_ACP_CA6-VSMD_Vertical, symbol Device:R_Potentiometer_US
- added SW2, SW3, SW4, SW5, SW6: SW_Push, Button_Switch_SMD:SW_SPST_PTS645, symbol Switch:SW_Push
- added U5: 74HC00, Package_DIP:DIP-14_W7.62mm, symbol 74xx:74HC00
- C1: footprint (none) -> Capacitor_SMD:CP_Elec_3x5.3
- R1, R2: footprint (none) -> Resistor_SMD:R_0201_0603Metric
- SW1: footprint (none) -> Button_Switch_SMD:SW_SPST_PTS645
- U1: value W65C02SxP -> W65C02S
- U2: footprint (none) -> Package_DIP:DIP-28_W15.24mm
- U3: value CY62256-70PC -> 62256
- U4: value W65C22NxP -> W65C22
Connections:
- net +5V: now also U4.20 (VCC), C2.1, C3.1, C4.1, DS1.16 (LEDK), DS1.2 (VDD), R3.1, R4.1, R5.1, R6.1, R7.1
- net GND: now also U4.1 (VSS), C2.2, C3.2, C4.2, DS1.1 (VSS), DS1.15 (LEDA), RV1.1, SW2.2, SW3.2, SW4.2, SW5.2, SW6.2
- net a0: now also U4.38 (RS0)
- net a1: now also U4.37 (RS1)
- net a13: now also U4.24 (CS1)
- net a14: now also U5.4
- net a15: now also U5.12, U5.13
- net a2: now also U4.36 (RS2)
- net a3: now also U4.35 (RS3)
- net at C1.1, R1.2, SW1.2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: now also U4.34 (~{RES})
- net at U1.37 (ϕ0), X1.8 (OUT): now also U4.25 (ϕ2), U5.9
- net at U4.10 (PB0): now also DS1.7 (DB0)
- net at U4.11 (PB1): now also DS1.8 (DB1)
- net at U4.12 (PB2): now also DS1.9 (DB2)
- net at U4.13 (PB3): now also DS1.10 (DB3)
- net at U4.14 (PB4): now also DS1.11 (DB4)
- net at U4.15 (PB5): now also DS1.12 (DB5)
- net at U4.16 (PB6): now also DS1.13 (DB6)
- net at U4.17 (PB7): now also DS1.14 (DB7)
- net at U4.2 (PA0): now also R3.2, SW2.1
- net at U4.21 (~{IRQ}): now also U1.4 (~{IRQ})
- net at U4.22 (R/~{W}): now also U1.34 (R/~{W})
- net at U4.23 (~{CS2}): now also U5.6
- net at U4.3 (PA1): now also R4.2, SW3.1
- net at U4.4 (PA2): now also R5.2, SW4.1
- net at U4.5 (PA3): now also R6.2, SW5.1
- net at U4.6 (PA4): now also R7.2, SW6.1
- net at U4.7 (PA5): now also DS1.6 (E)
- net at U4.8 (PA6): now also DS1.5 (R/~{W})
- net at U4.9 (PA7): now also DS1.4 (RS)
- net at U3.20 (~{CS}): now also U5.8
- net at U2.20 (~{CS}): now also U5.10, U5.11, U5.5
- new net: DS1.3 (Vo), RV1.2
- no-connect marks 6 -> 10

Commit message: bumb
Parts:
- DS1: footprint Display:HY1602E -> Display:WC1602A
Other:
- note added: "apparently I need these"
- note added: "switches for user input if I code that somehow"
Changed lines of the file:
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@@
     (stroke (width 0) (type default))
+  )
+  (text "switches for user input if I code that somehow" (at 223.52 58.42 0)
+    (effects (font (size 1.27 1.27)) (justify left bottom))
+  )
+  (text "apparently I need these" (at 25.4 110.49 0)
+    (effects (font (size 1.27 1.27)) (justify left bottom))
   )
   (label "a0" (at 140.97 50.8 0) (fields_autoplaced)
@@
       (effects (font (size 1.27 1.27)) (justify left))
     )
-    (property "Footprint" "Display:HY1602E" (at 234.95 109.22 0)
+    (property "Footprint" "Display:WC1602A" (at 234.95 109.22 0)
       (effects (font (size 1.27 1.27) italic) hide)
     )

Commit message: Add files via upload
Parts:
- DS1: value HY1602E -> HD44780U
Connections:
- no-connect marks 10 -> 11
Changed lines of the file:
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@@
   (no_connect (at 46.99 90.17))
   (no_connect (at 46.99 97.79))
+  (no_connect (at 251.46 67.31))
   (no_connect (at 46.99 92.71))
   (no_connect (at 46.99 62.23))
@@
       (effects (font (size 1.27 1.27)) (justify left))
     )
-    (property "Value" "HY1602E" (at 237.1441 66.04 0)
+    (property "Value" "HD44780U" (at 237.1441 66.04 0)
       (effects (font (size 1.27 1.27)) (justify left))
     )
@@
         (path "/28248d1b-65d0-4e2e-a100-551a14ee840a"
           (reference "#PWR019") (unit 1)
-        )
-      )
-    )
-  )
-  (symbol (lib_id "power:+5V") (at 234.95 66.04 0) (unit 1)
-    (in_bom yes) (on_board yes) (dnp no) (fields_autoplaced)
-    (property "Reference" "#PWR017" (at 234.95 69.85 0)
-      (effects (font (size 1.27 1.27)) hide)
-    )
-    (property "Value" "+5V" (at 234.95 60.96 0)
-      (effects (font (size 1.27 1.27)))
-    )
-    (property "Footprint" "" (at 234.95 66.04 0)
-      (effects (font (size 1.27 1.27)) hide)
-    )
-    (property "Datasheet" "" (at 234.95 66.04 0)
-      (effects (font (size 1.27 1.27)) hide)
-    )
-    (pin "1")
-    (instances
-      (project "6502 PCB"
-        (path "/28248d1b-65d0-4e2e-a100-551a14ee840a"
-          (reference "#PWR017") (unit 1)
         )
       )
@@
         )
       )
+    )
+  )
+  (symbol (lib_id "power:+5V") (at 234.95 66.04 0) (unit 1)
+    (in_bom yes) (on_board yes) (dnp no) (fields_autoplaced)
+    (property "Reference" "#PWR017" (at 234.95 69.85 0)
+      (effects (font (size 1.27 1.27)) hide)
+    )
+    (property "Value" "+5V" (at 234.95 60.96 0)
+      (effects (font (size 1.27 1.27)))
+    )
+    (property "Footprint" "" (at 234.95 66.04 0)
+      (effects (font (size 1.27 1.27)) hide)
+    )
+    (property "Datasheet" "" (at 234.95 66.04 0)
+      (effects (font (size 1.27 1.27)) hide)
+    )
+    (pin "1")
+    (instances
+      (project "6502 PCB"
+        (path "/28248d1b-65d0-4e2e-a100-551a14ee840a"
+          (reference "#PWR017") (unit 1)
+        )
+      )

Commit message: aaaaaaaaaaaaaaaaaaaa
Parts:
- DS1: footprint Display:WC1602A -> Display:HY1602E
Connections:
- net +5V: now also DS1.1 (LEDK), DS1.4 (VDD); no longer DS1.16 (LEDK), DS1.2 (VDD)
- net GND: now also DS1.2 (LEDA), DS1.3 (VSS); no longer DS1.1 (VSS), DS1.15 (LEDA)
- net at DS1.10 (DB1): now also U4.11 (PB1); no longer U4.13 (PB3)
- net at DS1.11 (DB2): now also U4.12 (PB2); no longer U4.14 (PB4)
- net at DS1.12 (DB3): now also U4.13 (PB3); no longer U4.15 (PB5)
- net at DS1.13 (DB4): now also U4.14 (PB4); no longer U4.16 (PB6)
- net at DS1.14 (DB5): now also U4.15 (PB5); no longer U4.17 (PB7)
- net at RV1.2: now also DS1.5 (Vo); no longer DS1.3 (Vo)
- net at U4.9 (PA7): now also DS1.6 (RS); no longer DS1.4 (RS)
- net at U4.8 (PA6): now also DS1.7 (R/~{W}); no longer DS1.5 (R/~{W})
- net at U4.7 (PA5): now also DS1.8 (E); no longer DS1.6 (E)
- net at U4.10 (PB0): now also DS1.9 (DB0); no longer DS1.7 (DB0)
- new net: DS1.15 (DB6), U4.16 (PB6)
- new net: DS1.16 (DB7), U4.17 (PB7)
Other:
- moved on the sheet: U3

Commit message: Add files via upload
Parts:
- removed C2, C3, C4: 0.1uf, Capacitor_SMD:CP_Elec_3x5.3, symbol Device:C
- removed R1, R2, R3, R4, R5, R6, R7: 1K, Resistor_SMD:R_0201_0603Metric, symbol Device:R
- added J1: power_source, TerminalBlock:TerminalBlock_Altech_AK300-2_P5.00mm, symbol Connector:Screw_Terminal_01x02
- added R1, R2, R3, R4, R5, R6, R7: 1K, Resistor_SMD:R_0201_0603Metric_Pad0.64x0.40mm_HandSolder, symbol Device:R_US
- DS1: footprint Display:HY1602E -> Display:WC1602A; symbol Display_Character:HY1602E -> HD44780U:HD44780U
Connections:
- net GND: now also DS1.1 (VSS), DS1.15 (LEDA), SW1.2, J1.1 (Pin_1); no longer DS1.2 (LEDA), DS1.3 (VSS), SW1.1
- net at SW6.1, U4.6 (PA4): now also R7.1
- net at SW3.1, U4.3 (PA1): now also R4.1
- net at U1.2 (RDY): now also R2.2
- net at SW4.1, U4.4 (PA2): now also R5.1
- net at SW5.1, U4.5 (PA3): now also R6.1
- net at DS1.10 (D3): now also U4.13 (PB3); no longer U4.11 (PB1)
- net at DS1.11 (D4): now also U4.14 (PB4); no longer U4.12 (PB2)
- net at DS1.12 (D5): now also U4.15 (PB5); no longer U4.13 (PB3)
- net at DS1.13 (D6): now also U4.16 (PB6); no longer U4.14 (PB4)
- net at DS1.14 (D7): now also U4.17 (PB7); no longer U4.15 (PB5)
- net VDD: now reaches DS1.16 (LEDK)
- net VDD: now also DS1.2 (VDD), U1.36 (BE), U1.6 (~{NMI}), U1.8 (VDD), U2.27 (~{WE}), U2.28 (VCC), U3.27 (~{WE}), U3.28 (VCC), U4.20 (VCC), X1.14 (Vcc), J1.2 (Pin_2), R1.1, R2.1, R3.2, R4.2, R5.2, R6.2, R7.2; no longer U4.17 (PB7)
- net at RV1.2: now also DS1.3 (V0); no longer DS1.5 (Vo)
- net at U4.9 (PA7): now also DS1.4 (RS); no longer DS1.6 (RS)
- net at U4.8 (PA6): now also DS1.5 (R/~{W}); no longer DS1.7 (R/~{W})
- net at U4.7 (PA5): now also DS1.6 (E); no longer DS1.8 (E)
- net at U4.10 (PB0): now also DS1.7 (D0); no longer DS1.9 (DB0)
- net at C1.1, U1.40 (~{RES}), U4.34 (~{RES}): now also SW1.1, R1.2; no longer SW1.2
- net at SW2.1, U4.2 (PA0): now also R3.1
- removed net +5V: DS1.1 (LEDK), DS1.4 (VDD), U1.36 (BE), U1.6 (~{NMI}), U1.8 (VDD), U2.27 (~{WE}), U2.28 (VCC), U3.27 (~{WE}), U3.28 (VCC), U4.20 (VCC), X1.14 (Vcc)
- new net: DS1.8 (D1), U4.11 (PB1)
- new net: DS1.9 (D2), U4.12 (PB2)
Other:
- note removed: "apparently I need these"
- moved on the sheet: C1, SW1

Commit message: pretty much done
Parts:
- removed DS1: HD44780U, Display:WC1602A, symbol HD44780U:HD44780U
- removed R4, R5, R6, R7: 1K, Resistor_SMD:R_0201_0603Metric_Pad0.64x0.40mm_HandSolder, symbol Device:R_US
- removed RV1: 10K, Potentiometer_SMD:Potentiometer_ACP_CA6-VSMD_Vertical, symbol Device:R_Potentiometer_US
- removed SW2, SW3, SW4, SW5, SW6: SW_Push, Button_Switch_SMD:SW_SPST_PTS645, symbol Switch:SW_Push
- added D1: LED, LED_SMD:LED_0201_0603Metric_Pad0.64x0.40mm_HandSolder, symbol Device:LED
- added J2, J3: Conn_01x08_Pin, Connector_PinHeader_1.00mm:PinHeader_1x08_P1.00mm_Vertical, symbol Connector:Conn_01x08_Pin
- C1: footprint Capacitor_SMD:CP_Elec_3x5.3 -> Capacitor_SMD:C_0201_0603Metric_Pad0.64x0.40mm_HandSolder
Connections:
- net GND: now also R3.2
- net VDD: now also D1.2 (A); no longer R3.2
- net at U4.4 (PA2): now also J2.3 (Pin_3)
- net at U4.3 (PA1): now also J2.2 (Pin_2)
- net at U4.13 (PB3): now also J3.4 (Pin_4)
- net at U4.14 (PB4): now also J3.5 (Pin_5)
- net at U4.15 (PB5): now also J3.6 (Pin_6)
- net at U4.16 (PB6): now also J3.7 (Pin_7)
- net at U4.17 (PB7): now also J3.8 (Pin_8)
- net at U4.9 (PA7): now also J2.8 (Pin_8)
- net at U4.8 (PA6): now also J2.7 (Pin_7)
- net at U4.7 (PA5): now also J2.6 (Pin_6)
- net at U4.10 (PB0): now also J3.1 (Pin_1)
- net at U4.11 (PB1): now also J3.2 (Pin_2)
- net at U4.12 (PB2): now also J3.3 (Pin_3)
- net at U4.2 (PA0): now also J2.1 (Pin_1); no longer R3.1
- net at U4.5 (PA3): now also J2.4 (Pin_4)
- net at U4.6 (PA4): now also J2.5 (Pin_5)
- new net: D1.1 (K), R3.1
- no-connect marks 11 -> 10
Other:
- note added: "Inputs"
- note added: "Outputs"
- note removed: "switches for user input if I code that somehow"

Commit message: Add files via upload
Parts:
- removed J2, J3: Conn_01x08_Pin, Connector_PinHeader_1.00mm:PinHeader_1x08_P1.00mm_Vertical, symbol Connector:Conn_01x08_Pin
- added J0, J10, J11, J12, J13, J14, J15, J16, J2, J3, J4, J5, J6, J7, J8, J9: Conn_01x01_Pin, Connector_PinHeader_1.00mm:PinHeader_1x01_P1.00mm_Vertical, symbol Connector:Conn_01x01_Pin
- C1: footprint Capacitor_SMD:C_0201_0603Metric_Pad0.64x0.40mm_HandSolder -> Capacitor_THT:C_Disc_D5.0mm_W2.5mm_P5.00mm
- D1: footprint LED_SMD:LED_0201_0603Metric_Pad0.64x0.40mm_HandSolder -> LED_THT:LED_D3.0mm
- R1, R2, R3: footprint Resistor_SMD:R_0201_0603Metric_Pad0.64x0.40mm_HandSolder -> Resistor_THT:R_Axial_DIN0204_L3.6mm_D1.6mm_P7.62mm_Horizontal
- SW1: footprint Button_Switch_SMD:SW_SPST_PTS645 -> Button_Switch_THT:SW_PUSH_6mm
Connections:
- net at U4.10 (PB0): now also J9.1 (Pin_1)
- net at U4.11 (PB1): now also J10.1 (Pin_1)
- net at U4.12 (PB2): now also J11.1 (Pin_1)
- net at U4.13 (PB3): now also J12.1 (Pin_1)
- net at U4.14 (PB4): now also J13.1 (Pin_1)
- net at U4.15 (PB5): now also J14.1 (Pin_1)
- net at U4.16 (PB6): now also J15.1 (Pin_1)
- net at U4.17 (PB7): now also J16.1 (Pin_1)
- net at U4.2 (PA0): now also J0.1 (Pin_1)
- net at U4.3 (PA1): now also J2.1 (Pin_1)
- net at U4.4 (PA2): now also J3.1 (Pin_1)
- net at U4.5 (PA3): now also J4.1 (Pin_1)
- net at U4.6 (PA4): now also J5.1 (Pin_1)
- net at U4.7 (PA5): now also J6.1 (Pin_1)
- net at U4.8 (PA6): now also J7.1 (Pin_1)
- net at U4.9 (PA7): now also J8.1 (Pin_1)

Commit message: pls work
Parts:
- removed J0, J10, J11, J12, J13, J14, J15, J16, J2, J3, J4, J5, J6, J7, J8, J9: Conn_01x01_Pin, Connector_PinHeader_1.00mm:PinHeader_1x01_P1.00mm_Vertical, symbol Connector:Conn_01x01_Pin
- added J17: Conn_01x16_Pin, Connector_PinHeader_2.00mm:PinHeader_1x16_P2.00mm_Vertical, symbol Connector:Conn_01x16_Pin
- J1: footprint TerminalBlock:TerminalBlock_Altech_AK300-2_P5.00mm -> TerminalBlock:TerminalBlock_bornier-2_P5.08mm
Connections:
- net at U4.2 (PA0): now also J17.1 (Pin_1)
- net at U4.5 (PA3): now also J17.4 (Pin_4)
- net at U4.13 (PB3): now also J17.12 (Pin_12)
- net at U4.12 (PB2): now also J17.11 (Pin_11)
- net at U4.14 (PB4): now also J17.13 (Pin_13)
- net at U4.17 (PB7): now also J17.16 (Pin_16)
- net at U4.7 (PA5): now also J17.6 (Pin_6)
- net at U4.6 (PA4): now also J17.5 (Pin_5)
- net at U4.16 (PB6): now also J17.15 (Pin_15)
- net at U4.9 (PA7): now also J17.8 (Pin_8)
- net at U4.10 (PB0): now also J17.9 (Pin_9)
- net at U4.3 (PA1): now also J17.2 (Pin_2)
- net at U4.11 (PB1): now also J17.10 (Pin_10)
- net at U4.15 (PB5): now also J17.14 (Pin_14)
- net at U4.4 (PA2): now also J17.3 (Pin_3)
- net at U4.8 (PA6): now also J17.7 (Pin_7)
Other:
- note removed: "Inputs"
- note removed: "Outputs"
