File: 6502 PCB.kicad_sch (KiCad schematic)
At the start: 18 parts, among them J1 Screw_Terminal_01x02, J2 Conn_01x16_Pin, SW1 RESET, U1 W65C02S, U2 28C256, U3 HM62256BLP, U4 74HC00, U5 WD65C22, X1 1MHz

Commit message: changed schematic a bunch
Parts:
- removed D1: LED, LED_THT:LED_D5.0mm, symbol Device:LED
- removed R3: 1k, Resistor_THT:R_Axial_DIN0207_L6.3mm_D2.5mm_P7.62mm_Horizontal, symbol Device:R_US
- removed R4: 3.3k, Resistor_THT:R_Axial_DIN0207_L6.3mm_D2.5mm_P7.62mm_Horizontal, symbol Device:R_US
- removed U2: 28C256, Package_DIP:DIP-28_W15.24mm, symbol Memory_EEPROM:28C256
- removed U3: HM62256BLP, Package_DIP:DIP-28_W15.24mm, symbol Memory_RAM:HM62256BLP
- removed U4: 74HC00, Package_DIP:DIP-14_W7.62mm, symbol 74xx:74HC00
- removed U5: WD65C22, Package_DIP:DIP-40_W15.24mm, symbol 65xx:WD65C22
- added J3: Conn_01x02_Pin, symbol Connector:Conn_01x02_Pin
- added U2: 74HC00, symbol 74xx:74HC00
- added U3: 28C256, symbol Memory_EEPROM:28C256
- added U4: 62256, Package_DIP:DIP-28_W15.24mm, symbol Memory_RAM:HM62256BLP
- added U5: WD65C22, Package_DIP:DIP-40_W15.24mm, symbol 6502_PCB:WD65C22
- C1: footprint Capacitor_THT:C_Disc_D3.0mm_W1.6mm_P2.50mm -> (none)
- C2, C3, C4: value 01.uF -> 0.1uF; footprint Capacitor_THT:C_Disc_D3.0mm_W1.6mm_P2.50mm -> (none)
- J1: footprint TerminalBlock:TerminalBlock_bornier-2_P5.08mm -> (none)
- J2: footprint Connector_PinSocket_2.54mm:PinSocket_1x16_P2.54mm_Vertical -> (none)
- R1, R2: footprint Resistor_THT:R_Axial_DIN0207_L6.3mm_D2.5mm_P7.62mm_Horizontal -> (none)
- SW1: footprint Button_Switch_THT:SW_PUSH_6mm -> (none)
Connections:
- net ~{RES} is gone; now on net ~{RESET}: C1.1, SW1.2, U1.40 (~{RES})
- net +5V: now also U1.36 (BE), J3.1 (Pin_1), U2.14 (VCC), U3.27 (~{WE}), U3.28 (VCC), U4.28 (VCC), U5.20 (VCC); no longer U1.38 (~{SO}), U1.4 (~{IRQ})
- net A0: now also U3.10 (A0), U5.38 (RS0)
- net A1: now also U3.9 (A1), U4.9 (A1), U5.37 (RS1)
- net A10: now also U3.21 (A10), U4.21 (A10)
- net A11: now also U3.23 (A11), U4.23 (A11)
- net A12: now also U3.2 (A12), U4.2 (A12)
- net A13: now also U3.26 (A13), U4.26 (A13), U5.24 (CS1)
- net A14: now also U2.4, U3.1 (A14), U4.1 (A14), U4.22 (~{OE})
- net A15: now also U2.12, U2.13
- net A2: now also U3.8 (A2), U4.8 (A2), U5.36 (RS2)
- net A3: now also U3.7 (A3), U4.7 (A3), U5.35 (RS3)
- net A4: now also U3.6 (A4), U4.6 (A4)
- net A5: now also U3.5 (A5), U4.5 (A5)
- net A6: now also U3.4 (A6), U4.4 (A6)
- net A7: now also U3.3 (A7), U4.3 (A7)
- net A8: now also U3.25 (A8), U4.25 (A8)
- net A9: now also U3.24 (A9), U4.24 (A9)
- net D0: now also U3.11 (D0), U4.11 (D0), U5.33 (D0)
- net D1: now also U3.12 (D1), U4.12 (D1), U5.32 (D1)
- net D2: now also U3.13 (D2), U4.13 (D2), U5.31 (D2)
- net D3: now also U3.15 (D3), U4.15 (D3), U5.30 (D3)
- net D4: now also U3.16 (D4), U4.16 (D4), U5.29 (D4)
- net D5: now also U3.17 (D5), U4.17 (D5), U5.28 (D5)
- net D6: now also U3.18 (D6), U4.18 (D6), U5.27 (D6)
- net D7: now also U3.19 (D7), U4.19 (D7), U5.26 (D7)
- net GND: now also J3.2 (Pin_2), U2.7 (GND), U3.14 (GND), U3.22 (~{OE}), U4.14 (GND), U5.1 (GND)
- net at J2.1 (Pin_1): now also U5.2 (PA0)
- net at J2.10 (Pin_10): now also U5.11 (PB1)
- net at J2.11 (Pin_11): now also U5.12 (PB2)
- net at J2.12 (Pin_12): now also U5.13 (PB3)
- net at J2.13 (Pin_13): now also U5.14 (PB4)
- net at J2.14 (Pin_14): now also U5.15 (PB5)
- net at J2.15 (Pin_15): now also U5.16 (PB6)
- net at J2.16 (Pin_16): now also U5.17 (PB7)
- net at J2.2 (Pin_2): now also U5.3 (PA1)
- net at J2.3 (Pin_3): now also U5.4 (PA2)
- net at J2.4 (Pin_4): now also U5.5 (PA3)
- net at J2.5 (Pin_5): now also U5.6 (PA4)
- net at J2.6 (Pin_6): now also U5.7 (PA5)
- net at J2.7 (Pin_7): now also U5.8 (PA6)
- net at J2.8 (Pin_8): now also U5.9 (PA7)
- net at J2.9 (Pin_9): now also U5.10 (PB0)
- net at R2.2: now also U1.2 (RDY); no longer U1.36 (BE)
- net ~{RESET}: now reaches R1.2
- net ~{RESET}: now also U5.34 (~{RESET}); no longer U1.2 (RDY)
- net PHI2 renamed CLK
- net CLK: now also U2.9, U5.25 (PHI2)
- net ~{RAMWE} renamed R/~{W}
- net R/~{W}: now also U4.27 (~{WE}), U5.22 (R/~{W})
- new net: U2.10, U2.11, U2.5, U3.20 (~{CS})
- new net: U2.8, U4.20 (~{CS})
- new net: U2.6, U5.23 (~{CS2})
- new net ~{IRQ}: U1.4 (~{IRQ}), U5.21 (~{IRQ})
- no-connect marks 12 -> 10
Other:
- note added: "Bypass capacitors Include at least on per power rail"

Commit message: finished PCB Design
Parts:
- added D1: LED, LED_THT:LED_D5.0mm_Clear, symbol Device:LED
- added R3: 1k, Resistor_THT:R_Axial_DIN0207_L6.3mm_D2.5mm_P10.16mm_Horizontal, symbol Device:R_US
- C1, C2, C3, C4: footprint (none) -> Capacitor_THT:C_Disc_D6.0mm_W2.5mm_P5.00mm
- J1: footprint (none) -> TerminalBlock_Phoenix:TerminalBlock_Phoenix_MKDS-1,5-2-5.08_1x02_P5.08mm_Horizontal
- J2: footprint (none) -> Connector_PinSocket_2.54mm:PinSocket_1x16_P2.54mm_Vertical
- J3: footprint (none) -> Connector_PinSocket_2.54mm:PinSocket_1x02_P2.54mm_Vertical
- R1, R2: footprint (none) -> Resistor_THT:R_Axial_DIN0207_L6.3mm_D2.5mm_P10.16mm_Horizontal
- SW1: footprint (none) -> Button_Switch_THT:SW_PUSH_6mm_H5mm
- U2: footprint (none) -> Package_DIP:DIP-14_W7.62mm
- U3: footprint (none) -> Package_DIP:DIP-28_W15.24mm
Connections:
- net +5V: now also R3.2
- net A0: now also U4.10 (A0)
- net GND: now also D1.1 (K)
- new net: D1.2 (A), R3.1
Changed lines of the file:
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@@
 		)
 	)
+	(label "A0"
+		(at 142.24 66.04 0)
+		(fields_autoplaced yes)
+		(effects
+			(font
+				(size 1.27 1.27)
+			)
+			(justify left bottom)
+		)
+	)
 	(label "D5"
 		(at 180.34 71.12 0)
@@
 	(global_label "+5V"
 		(shape input)
+		(at 120.65 168.91 90)
+		(fields_autoplaced yes)
+		(effects
+			(font
+				(size 1.27 1.27)
+			)
+			(justify left)
+		)
+		(property "Intersheetrefs" "${INTERSHEET_REFS}"
+			(at 120.65 162.0543 90)
+			(effects
+				(font
+					(size 1.27 1.27)
+				)
+				(justify left)
+				(hide yes)
+			)
+		)
+	)
+	(global_label "+5V"
+		(shape input)
 		(at 50.8 173.99 90)
 		(fields_autoplaced yes)
@@
 	(global_label "GND"
 		(shape input)
+		(at 120.65 184.15 270)
+		(fields_autoplaced yes)
+		(effects
+			(font
+				(size 1.27 1.27)
+			)
+			(justify right)
+		)
+		(property "Intersheetrefs" "${INTERSHEET_REFS}"
+			(at 120.65 191.0057 90)
+			(effects
+				(font
+					(size 1.27 1.27)
+				)
+				(justify right)
+				(hide yes)
+			)
+		)
+	)
+	(global_label "GND"
+		(shape input)
 		(at 50.8 181.61 270)
 		(fields_autoplaced yes)
@@
 			)
 		)
-		(property "Footprint" ""
+		(property "Footprint" "Resistor_THT:R_Axial_DIN0207_L6.3mm_D2.5mm_P10.16mm_Horizontal"
 			(at 44.704 37.084 90)
 			(effects
@@
 	)
 	(symbol
+		(lib_id "Device:R_US")
+		(at 120.65 172.72 180)
+		(unit 1)
+		(exclude_from_sim no)
+		(in_bom yes)
+		(on_board yes)
+		(dnp no)
+		(fields_autoplaced yes)
+		(property "Reference" "R3"
+			(at 123.19 171.4499 0)
+			(effects
+				(font
+					(size 1.27 1.27)
+				)
+				(justify right)
+			)
+		)
+		(property "Value" "1k"
+			(at 123.19 173.9899 0)
+			(effects
+				(font
+					(size 1.27 1.27)
+				)
+				(justify right)
+			)
+		)
+		(property "Footprint" "Resistor_THT:R_Axial_DIN0207_L6.3mm_D2.5mm_P10.16mm_Horizontal"
+			(at 119.634 172.466 90)
+			(effects
+				(font
+					(size 1.27 1.27)
+				)
+				(hide yes)
+			)
+		)
+		(property "Datasheet" "~"
+			(at 120.65 172.72 0)
+			(effects
+				(font
+					(size 1.27 1.27)
+				)
+				(hide yes)
+			)
+		)
+		(property "Description" "Resistor, US symbol"
+			(at 120.65 172.72 0)
+			(effects
+				(font
+					(size 1.27 1.27)
+				)
+				(hide yes)
+			)
+		)
+		(pin "2"
+		)
+		(pin "1"
+		)
+		(instances
+			(project "6502 PCB"
+				(path "/28248d1b-65d0-4e2e-a100-551a14ee840a"
+					(reference "R3")
+					(unit 1)
+				)
+			)
+		)
+	)
+	(symbol
 		(lib_id "Oscillator:ACO-xxxMHz")
 		(at 76.2 27.94 0)
@@
 			)
 		)
-		(property "Footprint" ""
+		(property "Footprint" "Connector_PinSocket_2.54mm:PinSocket_1x16_P2.54mm_Vertical"
 			(at 234.95 81.28 0)
 			(effects
@@
 			)
 		)
-		(property "Footprint" ""
+		(property "Footprint" "Capacitor_THT:C_Disc_D6.0mm_W2.5mm_P5.00mm"
 			(at 64.4652 48.26 0)
 			(effects
@@
 			)
 		)
-		(property "Footprint" ""
+		(property "Footprint" "Package_DIP:DIP-28_W15.24mm"
 			(at 107.95 88.9 0)
 			(effects
@@
 	)
 	(symbol
+		(lib_id "Device:LED")
+		(at 120.65 180.34 90)
+		(unit 1)
+		(exclude_from_sim no)
+		(in_bom yes)
+		(on_board yes)
+		(dnp no)
+		(fields_autoplaced yes)
+		(property "Reference" "D1"
+			(at 124.46 180.6574 90)
+			(effects
+				(font
+					(size 1.27 1.27)
+				)
+				(justify right)
+			)
+		)
+		(property "Value" "LED"
+			(at 124.46 183.1974 90)
+			(effects
+				(font
+					(size 1.27 1.27)
+				)
+				(justify right)
+			)
+		)
+		(property "Footprint" "LED_THT:LED_D5.0mm_Clear"
+			(at 120.65 180.34 0)
+			(effects
+				(font
+					(size 1.27 1.27)
+				)
+				(hide yes)
+			)
+		)
+		(property "Datasheet" "~"
+			(at 120.65 180.34 0)
+			(effects
+				(font
+					(size 1.27 1.27)
+				)
+				(hide yes)
+			)
+		)
+		(property "Description" "Light emitting diode"
+			(at 120.65 180.34 0)
+			(effects
+				(font
+					(size 1.27 1.27)
+				)
+				(hide yes)
+			)
+		)
+		(pin "1"
+		)
+		(pin "2"
+		)
+		(instances
+			(project ""
+				(path "/28248d1b-65d0-4e2e-a100-551a14ee840a"
+					(reference "D1")
+					(unit 1)
+				)
+			)
+		)
+	)
+	(symbol
 		(lib_id "W65C02S:W65C02S")
 		(at 57.15 99.06 0)
@@
 			)
 		)
-		(property "Footprint" ""
+		(property "Footprint" "Button_Switch_THT:SW_PUSH_6mm_H5mm"
 			(at 45.72 44.45 0)
 			(effects
@@
 			)
 		)
-		(property "Footprint" ""
+		(property "Footprint" "Package_DIP:DIP-14_W7.62mm"
 			(at 57.15 139.7 0)
 			(effects
@@
 			)
 		)
-		(property "Footprint" ""
+		(property "Footprint" "Package_DIP:DIP-14_W7.62mm"
 			(at 130.81 137.16 0)
 			(effects
@@
 			)
 		)
-		(property "Footprint" ""
+		(property "Footprint" "Package_DIP:DIP-14_W7.62mm"
 			(at 163.83 142.24 0)
 			(effects
@@
 			)
 		)
-		(property "Footprint" ""
+		(property "Footprint" "Capacitor_THT:C_Disc_D6.0mm_W2.5mm_P5.00mm"
 			(at 51.7652 181.61 0)
 			(effects
@@
 			)
 		)
-		(property "Footprint" ""
+		(property "Footprint" "Resistor_THT:R_Axial_DIN0207_L6.3mm_D2.5mm_P10.16mm_Horizontal"
 			(at 43.434 67.564 90)
 			(effects
@@
 			)
 		)
-		(property "Footprint" ""
+		(property "Footprint" "Package_DIP:DIP-14_W7.62mm"
 			(at 50.8 152.4 0)
 			(effects
@@
 			)
 		)
-		(property "Footprint" ""
+		(property "Footprint" "Capacitor_THT:C_Disc_D6.0mm_W2.5mm_P5.00mm"
 			(at 64.4652 181.61 0)
 			(effects
@@
 			)
 		)
-		(property "Footprint" ""
+		(property "Footprint" "Capacitor_THT:C_Disc_D6.0mm_W2.5mm_P5.00mm"
 			(at 39.0652 181.61 0)
 			(effects
@@
 			)
 		)
-		(property "Footprint" ""
+		(property "Footprint" "TerminalBlock_Phoenix:TerminalBlock_Phoenix_MKDS-1,5-2-5.08_1x02_P5.08mm_Horizontal"
 			(at 17.78 25.4 0)
 			(effects
@@
 			)
 		)
-		(property "Footprint" ""
+		(property "Footprint" "Connector_PinSocket_2.54mm:PinSocket_1x02_P2.54mm_Vertical"
 			(at 234.95 113.03 0)
 			(effects

Commit message: aaaaaaaaaaaaaaahhhhhhhhhhhhhhhhhhhhhhh
Parts:
- added J4: Conn_01x16_Pin, Connector_PinSocket_2.54mm:PinSocket_1x16_P2.54mm_Vertical, symbol Connector:Conn_01x16_Pin
- added J5: Conn_01x08_Pin, Connector_PinSocket_2.54mm:PinSocket_1x08_P2.54mm_Vertical, symbol Connector:Conn_01x08_Pin
Connections:
- net A0: now also J4.1 (Pin_1)
- net A1: now also J4.2 (Pin_2)
- net A10: now also J4.11 (Pin_11)
- net A11: now also J4.12 (Pin_12)
- net A12: now also J4.13 (Pin_13)
- net A13: now also J4.14 (Pin_14)
- net A14: now also J4.15 (Pin_15)
- net A15: now also J4.16 (Pin_16)
- net A2: now also J4.3 (Pin_3)
- net A3: now also J4.4 (Pin_4)
- net A4: now also J4.5 (Pin_5)
- net A5: now also J4.6 (Pin_6)
- net A6: now also J4.7 (Pin_7)
- net A7: now also J4.8 (Pin_8)
- net A8: now also J4.9 (Pin_9)
- net A9: now also J4.10 (Pin_10)
- net D0: now also J5.1 (Pin_1)
- net D1: now also J5.2 (Pin_2)
- net D2: now also J5.3 (Pin_3)
- net D3: now also J5.4 (Pin_4)
- net D4: now also J5.5 (Pin_5)
- net D5: now also J5.6 (Pin_6)
- net D6: now also J5.7 (Pin_7)
- net D7: now also J5.8 (Pin_8)
